Commit message: Fix build

File: urdf/separate_model.xacro (robot description, xacro)
@@ -13,5 +13,5 @@
       <origin xyz="0 0 0" rpy="0 0 0" />
       <geometry>
-      <mesh filename="package://efr_pacsim/urdf/Model_without_Steering_Tires.stl" scale="0.01 0.01 0.01"/>
+      <mesh filename="package://pacsim/urdf/Model_without_Steering_Tires.stl" scale="0.01 0.01 0.01"/>
       </geometry>
     </visual>
@@ -21,5 +21,5 @@
       <origin rpy="0.0 0 0" xyz="0 0 0"/>
       <geometry>
-      <mesh filename="package://efr_pacsim/urdf/FL_Inside.stl" scale="0.01 0.01 0.01"/>
+      <mesh filename="package://pacsim/urdf/FL_Inside.stl" scale="0.01 0.01 0.01"/>
       </geometry>
       </visual>
@@ -29,5 +29,5 @@
       <origin rpy="0.0 0 0" xyz="0 0 0"/>
       <geometry>
-      <mesh filename="package://efr_pacsim/urdf/FL_Outside.stl" scale="0.01 0.01 0.01"/>
+      <mesh filename="package://pacsim/urdf/FL_Outside.stl" scale="0.01 0.01 0.01"/>
       </geometry>
     </visual>
@@ -37,5 +37,5 @@
       <origin rpy="0.0 0 0" xyz="0 0 0"/>
       <geometry>
-      <mesh filename="package://efr_pacsim/urdf/FR_Inside.stl" scale="0.01 0.01 0.01"/>
+      <mesh filename="package://pacsim/urdf/FR_Inside.stl" scale="0.01 0.01 0.01"/>
       </geometry>
       </visual>
@@ -45,5 +45,5 @@
       <origin rpy="0.0 0 3.1415" xyz="0 0 0"/>
       <geometry>
-      <mesh filename="package://efr_pacsim/urdf/FL_Outside.stl" scale="0.01 0.01 0.01"/>
+      <mesh filename="package://pacsim/urdf/FL_Outside.stl" scale="0.01 0.01 0.01"/>
       </geometry>
     </visual>
@@ -53,5 +53,5 @@
       <origin rpy="0.0 0 0" xyz="0 0 0"/>
       <geometry>
-      <mesh filename="package://efr_pacsim/urdf/RR_Inside.stl" scale="0.01 0.01 0.01"/>
+      <mesh filename="package://pacsim/urdf/RR_Inside.stl" scale="0.01 0.01 0.01"/>
       </geometry>
       </visual>
@@ -61,5 +61,5 @@
       <origin rpy="0.0 0 3.14" xyz="0 0 0"/>
       <geometry>
-      <mesh filename="package://efr_pacsim/urdf/FL_Outside.stl" scale="0.01 0.01 0.01"/>
+      <mesh filename="package://pacsim/urdf/FL_Outside.stl" scale="0.01 0.01 0.01"/>
       </geometry>
     </visual>
@@ -69,5 +69,5 @@
       <origin rpy="0.0 0 3.1415" xyz="0 0 0"/>
       <geometry>
-      <mesh filename="package://efr_pacsim/urdf/RR_Inside.stl" scale="0.01 0.01 0.01"/>
+      <mesh filename="package://pacsim/urdf/RR_Inside.stl" scale="0.01 0.01 0.01"/>
       </geometry>
       </visual>
@@ -77,5 +77,5 @@
       <origin rpy="0.0 0 0" xyz="0 0 0"/>
       <geometry>
-      <mesh filename="package://efr_pacsim/urdf/FL_Outside.stl" scale="0.01 0.01 0.01"/>
+      <mesh filename="package://pacsim/urdf/FL_Outside.stl" scale="0.01 0.01 0.01"/>
       </geometry>
     </visual>
@@ -85,5 +85,5 @@
       <origin rpy="0.0 0 0" xyz="0 0 0"/>
       <geometry>
-      <mesh filename="package://efr_pacsim/urdf/Steering_Wheel.stl" scale="0.01 0.01 0.01"/>
+      <mesh filename="package://pacsim/urdf/Steering_Wheel.stl" scale="0.01 0.01 0.01"/>
       </geometry>
     </visual>

Commit message: fix: fixed car showing up weird in Foxglove and steering being in the actuator

File: urdf/separate_model.xacro (robot description, xacro)
@@ -11,5 +11,5 @@
    <link name="Modell">
     <visual>
-      <origin xyz="0 0 0" rpy="0 0 0" />
+      <origin xyz="0 0 0" rpy="-1.57 0 0" />
       <geometry>
       <mesh filename="package://pacsim/urdf/Model_without_Steering_Tires.stl" scale="0.01 0.01 0.01"/>
@@ -19,5 +19,5 @@
   <link name="FL_inside">
     <visual>
-      <origin rpy="0.0 0 0" xyz="0 0 0"/>
+      <origin rpy="-1.57 0 0" xyz="0 0 0"/>
       <geometry>
       <mesh filename="package://pacsim/urdf/FL_Inside.stl" scale="0.01 0.01 0.01"/>
@@ -27,5 +27,5 @@
   <link name="FL_outside">
     <visual>
-      <origin rpy="0.0 0 0" xyz="0 0 0"/>
+      <origin rpy="-1.57 0 0" xyz="0 0 0"/>
       <geometry>
       <mesh filename="package://pacsim/urdf/FL_Outside.stl" scale="0.01 0.01 0.01"/>
@@ -35,5 +35,5 @@
   <link name="FR_inside">
     <visual>
-      <origin rpy="0.0 0 0" xyz="0 0 0"/>
+      <origin rpy="-1.57 0 0" xyz="0 0 0"/>
       <geometry>
       <mesh filename="package://pacsim/urdf/FR_Inside.stl" scale="0.01 0.01 0.01"/>
@@ -43,5 +43,5 @@
   <link name="FR_outside">
     <visual>
-      <origin rpy="0.0 0 3.1415" xyz="0 0 0"/>
+      <origin rpy="-1.57 0 3.1415" xyz="0 0 0"/>
       <geometry>
       <mesh filename="package://pacsim/urdf/FL_Outside.stl" scale="0.01 0.01 0.01"/>
@@ -51,5 +51,5 @@
   <link name="RR_inside">
     <visual>
-      <origin rpy="0.0 0 0" xyz="0 0 0"/>
+      <origin rpy="-1.57 0 0" xyz="0 0 0"/>
       <geometry>
       <mesh filename="package://pacsim/urdf/RR_Inside.stl" scale="0.01 0.01 0.01"/>
@@ -59,5 +59,5 @@
   <link name="RR_outside">
     <visual>
-      <origin rpy="0.0 0 3.14" xyz="0 0 0"/>
+      <origin rpy="-1.57 0 3.14" xyz="0 0 0"/>
       <geometry>
       <mesh filename="package://pacsim/urdf/FL_Outside.stl" scale="0.01 0.01 0.01"/>
@@ -67,5 +67,5 @@
   <link name="RL_inside">
     <visual>
-      <origin rpy="0.0 0 3.1415" xyz="0 0 0"/>
+      <origin rpy="-1.57 0 3.1415" xyz="0 0 0"/>
       <geometry>
       <mesh filename="package://pacsim/urdf/RR_Inside.stl" scale="0.01 0.01 0.01"/>
@@ -75,5 +75,5 @@
   <link name="RL_outside">
     <visual>
-      <origin rpy="0.0 0 0" xyz="0 0 0"/>
+      <origin rpy="-1.57 0 0" xyz="0 0 0"/>
       <geometry>
       <mesh filename="package://pacsim/urdf/FL_Outside.stl" scale="0.01 0.01 0.01"/>

Commit message: fixNamingforJoints

File: urdf/separate_model.xacro (robot description, xacro)
@@ -120,9 +120,10 @@
     <axis xyz="0 1 0" />
   </joint>
-  <joint name="RR_inside" type="fixed">
+  <joint name="RR_steer" type="revolute">
     <parent link="Modell"/>
     <child link="RR_inside"/>
     <origin xyz="-1.64 -0.58 0.204" rpy="0 0 0" />
     <axis xyz="0 0 1" />
+    <limit upper=".5" lower="-.5" effort="10" velocity="10" />
   </joint>
   <joint name="RR_rotate" type="continuous">
@@ -132,9 +133,10 @@
     <axis xyz="0 1 0" />
   </joint>
-  <joint name="RL_inside" type="fixed">
+  <joint name="RL_steer" type="revolute">
     <parent link="Modell"/>
     <child link="RL_inside"/>
     <origin xyz="-1.64 0.58 0.204" rpy="0 0 0" />
     <axis xyz="0 0 1" />
+    <limit upper=".5" lower="-.5" effort="10" velocity="10" />
   </joint>
   <joint name="RL_rotate" type="continuous">
